File: deltarobot.kicad_sch (KiCad schematic)
At the start: 59 parts, among them M1 Pomp, M2 Motor_Servo, M3 Motor_Servo, M4 Motor_Servo, P1 RFID-RC522, Q2 BC547, SW1 SW, SW10 SW, SW11 SW_Push, SW2 SW, SW3 SW, SW4 SW, SW5 SW, SW6 SW, SW7 SW, SW8 SW, SW9 SW, U1 L298N, U2 7805, U3 noodknop

Commit message: final version for print
Connections:
- net AX is gone; now on net A1: R11.1
- net +5V: now also A1.D7; no longer A1.D27, A1.D28, A1.D29, A1.D30, A1.D31, A1.D32, A1.D33, A1.D34, A1.D35, A1.D36, R12.1, R13.1, R14.1, R15.1, R16.1, R17.1, R18.1, R19.1, R20.1, R21.1, U1.5 (IN1), U1.7 (IN2)
- net A1: now reaches A1.A1
- net D15: now reaches A1.D14 (D14/TX3)
- net D15: now also U1.7 (IN2)
- net D14: now reaches A1.D15 (D15/RX3)
- net D14: now also U1.5 (IN1)
- removed net PWMX: A1.D12, A1.D13, A1.D22, M2.1 (PWM), M3.1 (PWM), M4.1 (PWM)
- new net D27: A1.D27, R12.1
- new net D28: A1.D28, R13.1
- new net D29: A1.D29, R14.1
- new net D30: A1.D30, R15.1
- new net D31: A1.D31, R16.1
- new net D32: A1.D32, R17.1
- new net D33: A1.D33, R18.1
- new net D34: A1.D34, R19.1
- new net D35: A1.D35, R20.1
- new net D36: A1.D36, R21.1
- new net PWM12: A1.D12, M2.1 (PWM)
- new net PWM13: A1.D13, M3.1 (PWM)
- new net PWM22: A1.D22, M4.1 (PWM)
- no-connect marks 67 -> 63
Other:
- note added: "schema's spuitbot"
- note removed: "schema's medispuitbot"
- moved on the sheet: A1, C1, D1, D10, D11, D12, D2, D3, D4, D5, D6, D7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
